File: InvertingAmplifier/Inverting Amplifier/Inverting Amplifier.kicad_pcb (KiCad board)
At the start: 2 copper layers, 6 parts, among them J1 Vin, J2 Vo, J3 Power, U1 LM741

Commit message: Edge Cut
Other:
- board outline added: 33 x 15.2 mm
